File: Hardware/Logger/DataProcessing.sch (KiCad schematic (older format))
At the start: 4 parts, among them CN1 Conn_02x19_Odd_Even, CN10 Conn_02x19_Odd_Even, CN2 Conn_02x19_Odd_Even, CN7 Conn_02x19_Odd_Even

Commit message: fix #27, fix #30, fix #32
Connections:
- net labels added: 5V, CS_ESP, ESP_ENABLE, ESP_FLASH_MODE, ESP_RX, ESP_TX, KEY_DOWN, KEY_LEFT, KEY_RIGHT, KEY_UP, MISO, MOSI, SCK
- wire segments 304 -> 301
Other:
- note added: "Note all is done via nucleo32 board connected on the bottom of the PCB.\nOn the top of the PCB there are connectors to stack new shield."
- note removed: "connectors to stack new shield"
- note removed: "connectors to stm32 board"
- moved on the sheet: CN1, CN10, CN2, CN7
