File: Hardware/Logger/DataStorage.sch (KiCad schematic (older format))
At the start: 1 part, among them J6 SD_Card

Commit message: fix #38
Parts:
- removed J6: SD_Card, Connector_Card:microSD_HC_Hirose_DM3BT-DSF-PEJS, symbol Connector:SD_Card
- added C12, C13, C14: 330n, Capacitor_SMD:C_0402_1005Metric, symbol Device:C
- added J6: 112K-TAA0-RA1_ATTEND, Logger:104B-TAA0-R_ATTEND, symbol Logger:112K-TAA0-RA1_ATTEND
- added R13, R19, R20, R25, R26, R27: 10k, Resistor_SMD:R_0805_2012Metric, symbol Device:R
Connections:
- new net: J6.1 (DAT2), R27.2
- new net: J6.8 (DAT1), R13.2
- new net 3V3: C12.1, C13.1, C14.1, J6.4 (VDD), R13.1, R19.1, R20.1, R25.1, R26.1, R27.1
- new net CS_SD: J6.2 (CD/DAT3), R26.2
- new net GND: C12.2, C13.2, C14.2, J6.10 (SHELL2), J6.6 (VSS), J6.9 (SHELL1)
- new net MISO: J6.7 (DAT0), R19.2
- new net MOSI: J6.3 (CMD), R25.2
- new net SCK: J6.5 (CLK), R20.2
