File: Hardware/Logger/Logger.sch (KiCad schematic (older format))
At the start: 0 parts

Commit message: fix #27, fix #30, fix #32
Other:
- note added: "TODO\npower supply external\npower supply for lcd\nesp \nnucleo\nno copper under esp\nstqcked design"
- note removed: "TODO\npower supply external\npower supply for lcd\nesp \nnucleo\nno copper under esp"
Changed lines of the file:
@@
 $Descr A4 11693 8268
 encoding utf-8
-Sheet 1 6
+Sheet 1 7
 Title ""
 Date ""
@@
 $EndSheet
 Text Notes 3800 4000 0    71   ~ 14
-TODO\npower supply external\npower supply for lcd\nesp \nnucleo\nno copper under esp
+TODO\npower supply external\npower supply for lcd\nesp \nnucleo\nno copper under esp\nstqcked design
+$Sheet
+S 6900 3850 500  150
+U 6144CC5A
+F0 "PowerSupply" 50
+F1 "PowerSupply.sch" 50
+$EndSheet
 $EndSCHEMATC

Commit message: fix #38
Other:
- note added: "TODO\n\nno copper under esp\nmale pins on top layer"
- note removed: "TODO\npower supply external\npower supply for lcd\nesp \nnucleo\nno copper under esp\nstqcked design"
Changed lines of the file:
@@
 $EndSheet
 Text Notes 3800 4000 0    71   ~ 14
-TODO\npower supply external\npower supply for lcd\nesp \nnucleo\nno copper under esp\nstqcked design
+TODO\n\nno copper under esp\nmale pins on top layer
 $Sheet
 S 6900 3850 500  150
