File: Hardware/ProcessingAndStorage/Logger.kicad_sch (KiCad schematic)
At the start: 0 parts

Commit message: fix #148, fix #146, fix #151, fix #157
Other:
- note removed: "TODO male pins on top layer"
Changed lines of the file:
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@@
 	(generator_version "8.0")
 	(paper "A4")
-	(text "TODO\n\nmale pins on top layer"
-		(exclude_from_sim no)
-		(at 96.52 101.6 0)
-		(effects
-			(font
-				(size 1.8034 1.8034)
-				(thickness 0.3607)
-				(bold yes)
-			)
-			(justify left bottom)
-		)
-	)
-	(sheet
-		(at 207.01 62.23)
+	(sheet
+		(at 100.33 49.53)
 		(size 12.7 3.81)
 		(fields_autoplaced yes)
@@
 		)
 		(property "Sheetname" "DataStorage"
-			(at 207.01 61.5945 0)
+			(at 100.33 48.8945 0)
 			(effects
 				(font
@@
 		)
 		(property "Sheetfile" "DataStorage.kicad_sch"
-			(at 207.01 66.5485 0)
+			(at 100.33 53.8485 0)
 			(effects
 				(font
@@
 	)
 	(sheet
-		(at 173.99 74.93)
+		(at 67.31 62.23)
 		(size 12.7 3.81)
 		(fields_autoplaced yes)
@@
 		)
 		(property "Sheetname" "DataProcessing"
-			(at 173.99 74.2945 0)
+			(at 67.31 61.5945 0)
 			(effects
 				(font
@@
 		)
 		(property "Sheetfile" "DataProcessing.kicad_sch"
-			(at 173.99 79.2485 0)
+			(at 67.31 66.5485 0)
 			(effects
 				(font
@@
 	)
 	(sheet
-		(at 207.01 74.93)
+		(at 100.33 62.23)
 		(size 12.7 3.81)
 		(fields_autoplaced yes)
@@
 		)
 		(property "Sheetname" "UserInterface"
-			(at 207.01 74.2945 0)
+			(at 100.33 61.5945 0)
 			(effects
 				(font
@@
 		)
 		(property "Sheetfile" "UserInterface.kicad_sch"
-			(at 207.01 79.2485 0)
+			(at 100.33 66.5485 0)
 			(effects
 				(font
@@
 	)
 	(sheet
-		(at 144.78 74.93)
+		(at 38.1 62.23)
 		(size 12.7 3.81)
 		(fields_autoplaced yes)
@@
 		)
 		(property "Sheetname" "Acquisition"
-			(at 144.78 74.2945 0)
+			(at 38.1 61.5945 0)
 			(effects
 				(font
@@
 		)
 		(property "Sheetfile" "Acquisition.kicad_sch"
-			(at 144.78 79.2485 0)
+			(at 38.1 66.5485 0)
 			(effects
 				(font
@@
 	)
 	(sheet
-		(at 207.01 87.63)
+		(at 100.33 74.93)
 		(size 12.7 3.81)
 		(fields_autoplaced yes)
@@
 		)
 		(property "Sheetname" "WiFiInterface"
-			(at 207.01 86.9945 0)
+			(at 100.33 74.2945 0)
 			(effects
 				(font
@@
 		)
 		(property "Sheetfile" "WiFiInterface.kicad_sch"
-			(at 207.01 91.9485 0)
+			(at 100.33 79.2485 0)
 			(effects
 				(font
@@
 	)
 	(sheet
-		(at 175.26 97.79)
+		(at 68.58 85.09)
 		(size 12.7 3.81)
 		(fields_autoplaced yes)
@@
 		)
 		(property "Sheetname" "PowerSupply"
-			(at 175.26 97.1545 0)
+			(at 68.58 84.4545 0)
 			(effects
 				(font
@@
 		)
 		(property "Sheetfile" "PowerSupply.kicad_sch"
-			(at 175.26 102.1085 0)
-			(effects
-				(font
+			(at 68.58 89.4085 0)
+			(effects
+				(font
