File: Hardware/ProcessingAndStorage/UserInterface.kicad_sch (KiCad schematic)
At the start: 16 parts, among them Q5 Q_Photo_NPN, SW1 SW_Push, SW2 SW_Push, SW3 SW_Push, SW4 SW_Push, U2 ST7735S

Commit message: fix #148, fix #146, fix #151, fix #157
Parts:
- added C9: 330n, Capacitor_SMD:C_0805_2012Metric, symbol Device:C
Connections:
- net BACKGROUND_LIGHT_SENSOR: now also C9.1
- net GND: now also C9.2
Other:
- note added: "NOTE: Displays from different manufacturers have different reference points. Backlight level will be adjusted via PWM from the microcontroller. The jumper on 3V3 is for measuring power consumption."
- note added: "NOTE: Key debouncing will be handled in firmware. GPIO internal pull-ups are used instead of discrete resistors."
- note added: "NOTE: The phototransistor is used to adjust the brightness of the LCD via the microcontroller."
- note removed: "NOTE: 1/ Displays from different manufacturers have different points. 2/ backlight level will be adjusted via PWM from the microcontroller. 3/ Jumper on V3V is for measuring of power consumption. TODO: create correct footprint and recheck pinout."
- note removed: "NOTE: 1/ Key debouncing will be done in firmware. 2/ GPIO internall pullups are used instead of discrete resistors."
- note removed: "NOTE: phototransistor is used to adjust brightness of the LCD via microcontroller."
- moved on the sheet: C19, C20, JP2, Q5, R3, SW1, SW2, SW3, SW4, TP1, TP2, TP3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
