File: Hardware/ProcessingAndStorage/WiFiInterface.kicad_sch (KiCad schematic)
At the start: 18 parts, among them J10 Conn_01x06_Socket, J11 Conn_01x08_Socket, J9 Conn_01x08_Socket, U1 ESP-12E

Commit message: fix #148, fix #146, fix #151, fix #157
Parts:
- removed JP5: Jumper_2_Small_Open, Jumper:SolderJumper-2_P1.3mm_Open_TrianglePad1.0x1.5mm, symbol Jumper:Jumper_2_Small_Open
- removed R15: 470R, Resistor_SMD:R_0805_2012Metric, symbol Device:R
- added TP10, TP9: TestPoint, TestPoint:TestPoint_Pad_D1.5mm, symbol Connector:TestPoint
Connections:
- net ESP32_RX: now also TP9.1
- net ESP32_TX: now also TP10.1
Other:
- moved on the sheet: C15, C16, C17, C6, D2, J10, J11, J9, JP1, R13, R14, R17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
