File: Hardware/ProcessingAndStorage/DataStorage.kicad_sch (KiCad schematic)
At the start: 10 parts, among them J1 Micro_SD_Card_Det2, U3 LD1117S50TR_SOT223

Commit message: hw 4.1 pcb, ci rework
Parts:
- removed J1: Micro_SD_Card_Det2, Connector_Card:SD_TE_2041021, symbol Connector:Micro_SD_Card_Det2
- removed JP5: Jumper_2_Small_Open, Jumper:SolderJumper-2_P1.3mm_Open_TrianglePad1.0x1.5mm, symbol Jumper:Jumper_2_Small_Open
- added C13: 4u7, Capacitor_SMD:C_0805_2012Metric, symbol Device:C
- added D5, D6, D7, D8: PJGBLC03C_R1_00001, Diode_SMD:D_SOD-323F, symbol Device:D_TVS
- added J3: SD_Card_Receptacle, Connector_Card:SD_TE_2041021, symbol Connector:SD_Card_Receptacle
- added JP4: SolderJumper_2_Bridged, Jumper:SolderJumper-2_P1.3mm_Bridged_Pad1.0x1.5mm, symbol Jumper:SolderJumper_2_Bridged
- added R12: 47k, Resistor_SMD:R_0805_2012Metric, symbol Device:R
- added TP5, TP6, TP7: TestPoint, TestPoint:TestPoint_Pad_D1.5mm, symbol Connector:TestPoint
- R10, R7, R8: value 47R -> 47k
- R9: value 47R -> 22R
- U3: footprint Package_TO_SOT_SMD:SOT-223 -> Package_TO_SOT_SMD:SOT-223-3_TabPin2
Connections:
- net 5V: now also JP4.1 (A)
- net GND: now also C13.2, D5.1 (A1), D6.1 (A1), D7.1 (A1), D8.1 (A1), J3.3 (VSS), J3.6 (VSS)
- net GPIO_9: now also R7.1, D6.2 (A2), J3.1 (CD/DAT3); no longer R8.1
- net SPI1_MISO: now also D7.2 (A2), J3.7 (DAT0), R12.1; no longer R10.1
- net SPI1_MOSI: now also R10.1, D8.2 (A2), J3.2 (CMD); no longer R7.1
- net at R7.2: now also C11.1, R10.2, R8.2, U3.2 (VO), C13.1, J3.4 (VDD), R12.2, TP7.1
- net at C10.1, C12.1, U3.3 (VI): now also JP4.2 (B)
- net at R9.2: now also R8.1, D5.2 (A2), J3.5 (CLK)
- new net: J3.11 (WRITE_PROTECT), TP6.1
- new net: J3.10 (CARD_DETECT), TP5.1
Other:
- note removed: "NOTE: Resistors in series with the SPI pins of the microSD are used for ESD protection. The jumper on 3V3 is for measuring power consumption."
- moved on the sheet: C10, C11, C12, R9, U3

Commit message: hw 4.1 integration
Parts:
- R8: value 47k -> 10k
Changed lines of the file:
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@@
 			)
 		)
-		(property "Value" "47k"
+		(property "Value" "10k"
 			(at 105.41 58.4199 0)
 			(effects
