File: Hardware/ProcessingAndStorage/ProcessingAndStorage.kicad_pcb (KiCad board)
At the start: 2 copper layers, 85 x 60 mm, 31 parts, among them J1 Micro_SD_Card_Det2, J5 Conn_02x11_Odd_Even, SW2 SW_SPDT_XKB_DMx-xxxx-1, U1 LD1117S50TR_SOT223, U2 ESP-12E, U3 LD1117S50TR_SOT223

Commit message: hw 4.1 pcb, ci rework
Parts:
- removed J5: Conn_02x11_Odd_Even, Connector_PinHeader_2.54mm:PinHeader_2x11_P2.54mm_Vertical
- removed JP5: Jumper_2_Small_Open, Jumper:SolderJumper-2_P1.3mm_Open_TrianglePad1.0x1.5mm
- removed SW2: SW_SPDT_XKB_DMx-xxxx-1, Button_Switch_THT:SW_Slide-03_Wuerth-WS-SLTV_10x2.5x6.4_P2.54mm
- added C13: 4u7, Capacitor_SMD:C_0805_2012Metric, F.Cu at (153.1, 98.9)
- added C18: 100n, Capacitor_SMD:C_0805_2012Metric, F.Cu at (177.2, 75.5)
- added C20: 100n, Capacitor_SMD:C_0805_2012Metric, F.Cu at (177.2, 72.0)
- added C9: 10u, Capacitor_SMD:C_0805_2012Metric, F.Cu at (175.1, 72.0)
- added D1: LED, LED_SMD:LED_0402_1005Metric, F.Cu at (199.2, 71.1)
- added D3: LED, LED_SMD:LED_0402_1005Metric, F.Cu at (213.6, 109.6)
- added D4: LED, LED_SMD:LED_0402_1005Metric, F.Cu at (201.4, 71.1)
- added D5: PJGBLC03C_R1_00001, Diode_SMD:D_SOD-323F, F.Cu at (155.4, 98.8)
- added D6: PJGBLC03C_R1_00001, Diode_SMD:D_SOD-323F, F.Cu at (145.6, 98.8)
- added D7: PJGBLC03C_R1_00001, Diode_SMD:D_SOD-323F, F.Cu at (160.6, 98.8)
- added D8: PJGBLC03C_R1_00001, Diode_SMD:D_SOD-323F, F.Cu at (148.2, 98.8)
- added J2: Conn_02x10_Odd_Even, Connector_PinHeader_2.54mm:PinHeader_2x10_P2.54mm_Horizontal, F.Cu at (204.3, 72.9)
- added J3: SD_Card_Receptacle, Connector_Card:SD_TE_2041021, F.Cu at (152.4, 84.0)
- added JP1: SolderJumper_2_Bridged, Jumper:SolderJumper-2_P1.3mm_Bridged_Pad1.0x1.5mm, F.Cu at (182.0, 91.1)
- added JP3: SolderJumper_2_Bridged, Jumper:SolderJumper-2_P1.3mm_Bridged_Pad1.0x1.5mm, F.Cu at (199.8, 82.2)
- added JP4: SolderJumper_2_Bridged, Jumper:SolderJumper-2_P1.3mm_Bridged_Pad1.0x1.5mm, F.Cu at (136.2, 109.8)
- added Q1: BC846, Package_TO_SOT_SMD:SOT-23, F.Cu at (197.4, 103.4)
- added Q2: BC846, Package_TO_SOT_SMD:SOT-23, F.Cu at (201.1, 103.4)
- added Q3: BC846, Package_TO_SOT_SMD:SOT-23, F.Cu at (191.8, 103.4)
- added Q4: BC846, Package_TO_SOT_SMD:SOT-23, F.Cu at (186.2, 103.4)
- added R11: 1k, Resistor_SMD:R_0805_2012Metric, F.Cu at (201.4, 73.9)
- added R12: 47k, Resistor_SMD:R_0805_2012Metric, F.Cu at (162.6, 98.9)
- added R17: 10k, Resistor_SMD:R_0805_2012Metric, F.Cu at (199.3, 108.5)
- added R18: 10k, Resistor_SMD:R_0805_2012Metric, F.Cu at (199.3, 106.4)
- added R20: 10k, Resistor_SMD:R_0805_2012Metric, F.Cu at (175.1, 75.5)
- added TP1: TestPoint, TestPoint:TestPoint_Pad_D1.5mm, F.Cu at (199.1, 91.1)
- added TP2: TestPoint, TestPoint:TestPoint_Pad_D1.5mm, F.Cu at (195.0, 94.7)
- added TP3: TestPoint, TestPoint:TestPoint_Pad_D1.5mm, F.Cu at (196.7, 92.6)
- added TP4: TestPoint, TestPoint:TestPoint_Pad_D1.5mm, F.Cu at (190.5, 97.8)
- added TP5: TestPoint, TestPoint:TestPoint_Pad_D1.5mm, F.Cu at (165.9, 99.3)
- added TP6: TestPoint, TestPoint:TestPoint_Pad_D1.5mm, F.Cu at (165.9, 102.9)
- added TP7: TestPoint, TestPoint:TestPoint_Pad_D1.5mm, F.Cu at (140.3, 98.3)
- added TP8: TestPoint, TestPoint:TestPoint_Pad_D1.5mm, F.Cu at (175.2, 91.8)
- added U4: ESP32-WROOM-32E, RF_Module:ESP32-WROOM-32D, F.Cu at (188.3, 79.1)
- C5: value 47u/6V3 -> 100n; footprint Capacitor_Tantalum_SMD:CP_EIA-3528-21_Kemet-B -> Capacitor_SMD:C_0805_2012Metric
- C7: value 100n -> 10u
- C8: value 470p -> 10u
- J1: value Micro_SD_Card_Det2 -> USB_B_Micro; footprint Connector_Card:SD_TE_2041021 -> HardwareDataLogger:USB_Micro-B_Molex-105017-0001_Extra_Mechanical_Pads
- R1: value 470R -> 10k
- R10, R7, R8: value 47R -> 47k
- R2, R3, R6: value 10k -> 1k
- R9: value 47R -> 22R
- U1, U3: footprint Package_TO_SOT_SMD:SOT-223 -> Package_TO_SOT_SMD:SOT-223-3_TabPin2
- U2: value ESP-12E -> CH340X; footprint RF_Module:ESP-12E -> Package_SO:MSOP-10_3x3mm_P0.5mm
- moved J1 68.8 mm to (210.0, 102.7), turned to 90 degrees
- moved D2 43.7 mm to (213.6, 108.5)
- moved C7 43.2 mm to (203.5, 109.5), turned to -90 degrees
- moved R1 40.4 mm to (209.8, 109.5), turned to 90 degrees
- moved C5 38.3 mm to (207.7, 109.5), turned to -90 degrees
- moved C6 36.0 mm to (205.6, 109.5), turned to -90 degrees
- moved U2 34.8 mm to (205.3, 104.5), turned to -90 degrees
- moved R3 32.9 mm to (186.8, 106.7)
- moved R5 30.1 mm to (189.0, 103.7), turned to 90 degrees
- moved R4 29.4 mm to (194.6, 103.7), turned to 90 degrees
- moved R2 27.6 mm to (192.0, 106.7), turned to 180 degrees
- moved C11 19.5 mm to (132.0, 107.4), turned to 180 degrees
- moved R6 19.2 mm to (199.2, 73.9), turned to -90 degrees
- moved R8 16.3 mm to (157.4, 98.9), turned to -90 degrees
- moved R9 15.6 mm to (157.2, 104.8), turned to 90 degrees
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Connections:
- C11 pad 1: Net-(J1-VDD) -> Net-(J3-VDD)
- C3 pad 1: 3V3 -> ESP_3V3
- C4 pad 1: 3V3 -> ESP_3V3
- C5 pad 1: ESP_PWR -> Net-(U2-V3)
- C6 pad 1: ESP_PWR -> ESP_3V3
- C7 pad 1: /WiFi/EN -> ESP_3V3
- C8 pad 1: NRST -> ESP_3V3
- D2 pad 2: /WiFi/GPIO13 -> ESP_3V3
- J1 pad 1: unconnected-(J1-DAT2-Pad1) -> Net-(J1-VBUS)
- J1 pad 2: Net-(J1-DAT3/CD) -> /SerialProgrammer/USB_N
- J1 pad 3: Net-(J1-CMD) -> /SerialProgrammer/USB_P
- J1 pad 4: Net-(J1-VDD) -> unconnected-(J1-ID-Pad4)
- J1 pad 5: Net-(J1-CLK) -> GND
- J6 pad 41: NRST -> unconnected-(J6-Pin_41-Pad41)
- J6 pad 43: BOOT0 -> unconnected-(J6-Pin_43-Pad43)
- R1 pad 1: Net-(D2-K) -> GND
- R1 pad 2: GND -> Net-(J1-VBUS)
- R10 pad 1: SPI1_MISO -> SPI1_MOSI
- R10 pad 2: Net-(J1-DAT0) -> Net-(J3-VDD)
- R2 pad 1: /WiFi/GPIO15 -> Net-(D2-K)
- R2 pad 2: GND -> Net-(Q3-C)
- R3 pad 1: ESP_PWR -> Net-(D3-K)
- R3 pad 2: /WiFi/GPIO2 -> Net-(Q4-C)
- R4 pad 1: ESP_PWR -> Net-(Q1-E)
- R4 pad 2: BOOT0 -> Net-(Q3-B)
- R5 pad 1: ESP_PWR -> Net-(Q2-E)
- R5 pad 2: /WiFi/EN -> Net-(Q4-B)
- R6 pad 1: ESP_PWR -> Net-(D1-K)
- R6 pad 2: NRST -> GND
- R7 pad 1: SPI1_MOSI -> GPIO_9
- R7 pad 2: Net-(J1-CMD) -> Net-(J3-VDD)
- R8 pad 1: GPIO_9 -> Net-(D5-A2)
- R8 pad 2: Net-(J1-DAT3/CD) -> Net-(J3-VDD)
- R9 pad 2: Net-(J1-CLK) -> Net-(D5-A2)
- U1 pad 2: 3V3 -> ESP_3V3
- U2 pad 1: NRST -> /SerialProgrammer/USB_P
- U2 pad 10: /WiFi/ESP32_MISO -> Net-(U2-V3)
- U2 pad 2: /WiFi/ESP_ADC -> /SerialProgrammer/USB_N
- U2 pad 3: /WiFi/EN -> GND
- U2 pad 4: /WiFi/GPIO16 -> Net-(Q1-E)
- U2 pad 5: /WiFi/GPIO14 -> unconnected-(U2-~{CTS}-Pad5)
- U2 pad 6: /WiFi/GPIO12 -> Net-(Q2-E)
- U2 pad 7: /WiFi/GPIO13 -> ESP_3V3
- U2 pad 8: ESP_PWR -> ESP_U0_TX
- U2 pad 9: /WiFi/ESP32_CS0 -> ESP_U0_RX
- U3 pad 2: Net-(J1-VDD) -> Net-(J3-VDD)
Routing:
- net ESP_3V3: track 0.00 -> 153.2 mm, vias 0 -> 1
- net NRST: track 95.4 -> 0.00 mm
- net ESP_PWR: track 75.6 -> 0.00 mm, vias 2 -> 0
- net Net-(J3-VDD): track 0.00 -> 64.0 mm, vias 0 -> 4
- net BOOT0: track 59.7 -> 0.00 mm, vias 2 -> 0
- net ESP_EN: track 0.00 -> 45.5 mm
- net ESP_U0_TX: track 0.00 -> 40.0 mm, vias 0 -> 2
- net ESP_U0_RX: track 0.00 -> 37.9 mm
- net USART1_TX: track 85.5 -> 52.4 mm, vias 2 -> 1
- net /WiFi/IO14: track 0.00 -> 32.7 mm, vias 0 -> 1
- net USART1_RX: track 87.5 -> 55.2 mm, vias 2 -> 1
- net /WiFi/IO26: track 0.00 -> 31.0 mm, vias 0 -> 1
- net /WiFi/EN: track 30.6 -> 0.00 mm
- net /WiFi/IO33: track 0.00 -> 30.2 mm, vias 0 -> 1
- net /WiFi/IO35: track 0.00 -> 30.0 mm, vias 0 -> 1
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Other:
- board size 85 x 60 mm -> 85 x 50 mm
- board text added: "J2 pins 23 22 21 19 18 VP VN VCC 34 35 32 33 25 26 27 14 13 04 GN GN"
- board text added: "ProcessingAndStorage rev 1.2"
- board text removed: "ProcessingAndStorage rev 1.0"

Commit message: hw 4.1 integration
Parts:
- R8: value 47k -> 10k
Changed lines of the file:
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@@
 			)
 		)
-		(property "Value" "47k"
+		(property "Value" "10k"
 			(at 0 1.65 90)
 			(layer "F.Fab")
