File: Hardware/ProcessingAndStorage/SerialProgrammer.kicad_sch (KiCad schematic)
At the start: 22 parts, among them J1 USB_B_Micro, Q1 BC846, Q2 BC846, Q3 BC846, Q4 BC846, U2 CH340X

Commit message: xx
Parts:
- J1: footprint Connector_USB:USB_Micro-B_Molex-105017-0001 -> HardwareDataLogger:USB_Micro-B_Molex-105017-0001_Extra_Mechanical_Pads
Connections:
- net USB+ renamed USB_P
- net USB- renamed USB_N
Other:
- moved on the sheet: C18, C5, C6, C7, D2, D3, J1, Q1, Q2, Q3, Q4, R1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

Commit message: hw 4.1 integration
Parts:
- added U5: CH340E, Package_SO:MSOP-10_3x3mm_P0.5mm, symbol Interface_USB:CH340E
Changed lines of the file:
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@@
+	)
+	(symbol
+		(lib_id "Interface_USB:CH340E")
+		(at 55.88 115.57 0)
+		(unit 1)
+		(exclude_from_sim no)
+		(in_bom yes)
+		(on_board yes)
+		(dnp no)
+		(fields_autoplaced yes)
+		(property "Reference" "U5"
+			(at 58.0233 130.81 0)
+			(effects
+				(font
+					(size 1.27 1.27)
+				)
+				(justify left)
+			)
+		)
+		(property "Value" "CH340E"
+			(at 58.0233 133.35 0)
+			(effects
+				(font
+					(size 1.27 1.27)
+				)
+				(justify left)
+			)
+		)
+		(property "Footprint" "Package_SO:MSOP-10_3x3mm_P0.5mm"
+			(at 57.15 129.54 0)
+			(effects
+				(font
+					(size 1.27 1.27)
+				)
+				(justify left)
+				(hide yes)
+			)
+		)
+		(property "Datasheet" "https://www.mpja.com/download/35227cpdata.pdf"
+			(at 46.99 95.25 0)
+			(effects
+				(font
+					(size 1.27 1.27)
+				)
+				(hide yes)
+			)
+		)
+		(property "Description" "USB serial converter, UART, MSOP-10"
+			(at 55.88 115.57 0)
+			(effects
+				(font
+					(size 1.27 1.27)
+				)
+				(hide yes)
+			)
+		)
+		(pin "2"
+		)
+		(pin "6"
+		)
+		(pin "7"
+		)
+		(pin "10"
+		)
+		(pin "8"
+		)
+		(pin "4"
+		)
+		(pin "1"
+		)
+		(pin "9"
+		)
+		(pin "5"
+		)
+		(pin "3"
+		)
+		(instances
+			(project ""
+				(path "/2dac91f6-5de1-492e-9a04-36ab71ef854f/097c6198-7414-46b7-a29c-2ab22bad5270"
+					(reference "U5")
+					(unit 1)
+				)
+			)
+		)
 	)
 	(symbol
