File: Hardware/MainBoard/MainBoard.kicad_sch (KiCad schematic)
At the start: 0 parts

Commit message: draft of mainboard
Other:
- sheet ModuleConnector renamed ModuleConnector1
- added sheet Breadboard (Breadboard.kicad_sch)
- added sheet Mechanic (Mechanic.kicad_sch)
- added sheet ModuleConnector2 (ModuleConnector2.kicad_sch)
- sheet ModuleConnector1: file ModuleConnector.kicad_sch -> ModuleConnector1.kicad_sch
Changed lines of the file:
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@@
+	)
+	(sheet
+		(at 119.38 101.6)
+		(size 12.7 3.81)
+		(fields_autoplaced yes)
+		(stroke
+			(width 0.1524)
+			(type solid)
+		)
+		(fill
+			(color 0 0 0 0.0000)
+		)
+		(property "Sheetname" "ModuleConnector2"
+			(at 119.38 100.8884 0)
+			(effects
+				(font
+					(size 1.27 1.27)
+				)
+				(justify left bottom)
+			)
+		)
+		(property "Sheetfile" "ModuleConnector2.kicad_sch"
+			(at 119.38 105.9946 0)
+			(effects
+				(font
+					(size 1.27 1.27)
+				)
+				(justify left top)
+			)
+		)
+		(instances
+			(project "MainBoard"
+				(path "/2dac91f6-5de1-492e-9a04-36ab71ef854f"
+					(page "5")
+				)
+			)
+		)
 	)
 	(sheet
@@
 			(color 0 0 0 0.0000)
 		)
-		(property "Sheetname" "ModuleConnector"
+		(property "Sheetname" "ModuleConnector1"
 			(at 114.3 84.3784 0)
 			(effects
@@
 			)
 		)
-		(property "Sheetfile" "ModuleConnector.kicad_sch"
+		(property "Sheetfile" "ModuleConnector1.kicad_sch"
 			(at 114.3 89.4846 0)
 			(effects
@@
 				)
 			)
+		)
+	)
+	(sheet
+		(at 63.5 125.73)
+		(size 12.7 3.81)
+		(fields_autoplaced yes)
+		(stroke
+			(width 0.1524)
+			(type solid)
+		)
+		(fill
+			(color 0 0 0 0.0000)
+		)
+		(property "Sheetname" "Breadboard"
+			(at 63.5 125.0184 0)
+			(effects
+				(font
+					(size 1.27 1.27)
+				)
+				(justify left bottom)
+			)
+		)
+		(property "Sheetfile" "Breadboard.kicad_sch"
+			(at 63.5 130.1246 0)
+			(effects
+				(font
+					(size 1.27 1.27)
+				)
+				(justify left top)
+			)
+		)
+		(property "Field2" ""
+			(at 63.5 125.73 0)
+			(effects
+				(font
+					(size 1.27 1.27)
+				)
+				(hide yes)
+			)
+		)
+		(instances
+			(project "MainBoard"
+				(path "/2dac91f6-5de1-492e-9a04-36ab71ef854f"
+					(page "6")
+				)
+			)
+		)
+	)
+	(sheet
+		(at 80.01 104.14)
+		(size 12.7 3.81)
+		(fields_autoplaced yes)
+		(stroke
+			(width 0.1524)
+			(type solid)
+		)
+		(fill
+			(color 0 0 0 0.0000)
+		)
+		(property "Sheetname" "Mechanic"
+			(at 80.01 103.4284 0)
+			(effects
+				(font
+					(size 1.27 1.27)
+				)
+				(justify left bottom)
+			)
+		)
+		(property "Sheetfile" "Mechanic.kicad_sch"
+			(at 80.01 108.5346 0)
+			(effects
+				(font
+					(size 1.27 1.27)
+				)
+				(justify left top)
+			)
+		)
+		(instances
+			(project "MainBoard"
+				(path "/2dac91f6-5de1-492e-9a04-36ab71ef854f"
+					(page "4")
+				)
+			)
