File: Hardware/MainBoard/MainBoard.kicad_sch (KiCad schematic)
At the start: 0 parts

Commit message: pcb draft
Other:
- removed sheet Acquisition
- removed sheet DataProcessing
- removed sheet DataStorage
- removed sheet UserInterface
- removed sheet WiFiInterface
- added sheet Breadboard (Breadboard.kicad_sch)
- added sheet Mechanic (Mechanic.kicad_sch)
- added sheet ModuleConnector1 (ModuleConnector1.kicad_sch)
- added sheet ModuleConnector2 (ModuleConnector2.kicad_sch)
- note removed: "TODO male pins on top layer"
Changed lines of the file:
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@@
 	(generator_version "8.0")
 	(paper "A4")
-	(text "TODO\n\nmale pins on top layer"
-		(exclude_from_sim no)
-		(at 96.52 101.6 0)
-		(effects
-			(font
-				(size 1.8034 1.8034)
-				(thickness 0.3607)
-				(bold yes)
-			)
-			(justify left bottom)
-		)
-	)
 	(sheet
-		(at 207.01 62.23)
-		(size 12.7 3.81)
-		(fields_autoplaced yes)
-		(stroke
-			(width 0)
-			(type solid)
-		)
-		(fill
-			(color 0 0 0 0.0000)
-		)
-		(property "Sheetname" "DataStorage"
-			(at 207.01 61.5945 0)
-			(effects
-				(font
-					(size 1.27 1.27)
-				)
-				(justify left bottom)
-			)
-		)
-		(property "Sheetfile" "DataStorage.kicad_sch"
-			(at 207.01 66.5485 0)
-			(effects
-				(font
-					(size 1.27 1.27)
-				)
-				(justify left top)
-			)
-		)
-		(instances
-			(project "Logger"
-				(path "/2dac91f6-5de1-492e-9a04-36ab71ef854f"
-					(page "4")
-				)
-			)
-		)
-	)
-	(sheet
-		(at 173.99 74.93)
-		(size 12.7 3.81)
-		(fields_autoplaced yes)
-		(stroke
-			(width 0)
-			(type solid)
-		)
-		(fill
-			(color 0 0 0 0.0000)
-		)
-		(property "Sheetname" "DataProcessing"
-			(at 173.99 74.2945 0)
-			(effects
-				(font
-					(size 1.27 1.27)
-				)
-				(justify left bottom)
-			)
-		)
-		(property "Sheetfile" "DataProcessing.kicad_sch"
-			(at 173.99 79.2485 0)
-			(effects
-				(font
-					(size 1.27 1.27)
-				)
-				(justify left top)
-			)
-		)
-		(instances
-			(project "Logger"
-				(path "/2dac91f6-5de1-492e-9a04-36ab71ef854f"
-					(page "3")
-				)
-			)
-		)
-	)
-	(sheet
-		(at 207.01 74.93)
-		(size 12.7 3.81)
-		(fields_autoplaced yes)
-		(stroke
-			(width 0)
-			(type solid)
-		)
-		(fill
-			(color 0 0 0 0.0000)
-		)
-		(property "Sheetname" "UserInterface"
-			(at 207.01 74.2945 0)
-			(effects
-				(font
-					(size 1.27 1.27)
-				)
-				(justify left bottom)
-			)
-		)
-		(property "Sheetfile" "UserInterface.kicad_sch"
-			(at 207.01 79.2485 0)
-			(effects
-				(font
-					(size 1.27 1.27)
-				)
-				(justify left top)
-			)
-		)
-		(instances
-			(project "Logger"
-				(path "/2dac91f6-5de1-492e-9a04-36ab71ef854f"
-					(page "6")
-				)
-			)
-		)
-	)
-	(sheet
-		(at 144.78 74.93)
-		(size 12.7 3.81)
-		(fields_autoplaced yes)
-		(stroke
-			(width 0)
-			(type solid)
-		)
-		(fill
-			(color 0 0 0 0.0000)
-		)
-		(property "Sheetname" "Acquisition"
-			(at 144.78 74.2945 0)
-			(effects
-				(font
-					(size 1.27 1.27)
-				)
-				(justify left bottom)
-			)
-		)
-		(property "Sheetfile" "Acquisition.kicad_sch"
-			(at 144.78 79.2485 0)
-			(effects
-				(font
-					(size 1.27 1.27)
-				)
-				(justify left top)
-			)
-		)
-		(instances
-			(project "Logger"
-				(path "/2dac91f6-5de1-492e-9a04-36ab71ef854f"
-					(page "2")
-				)
-			)
-		)
-	)
-	(sheet
-		(at 207.01 87.63)
-		(size 12.7 3.81)
-		(fields_autoplaced yes)
-		(stroke
-			(width 0)
-			(type solid)
-		)
-		(fill
-			(color 0 0 0 0.0000)
-		)
-		(property "Sheetname" "WiFiInterface"
-			(at 207.01 86.9945 0)
-			(effects
-				(font
-					(size 1.27 1.27)
-				)
-				(justify left bottom)
-			)
-		)
-		(property "Sheetfile" "WiFiInterface.kicad_sch"
-			(at 207.01 91.9485 0)
-			(effects
-				(font
-					(size 1.27 1.27)
-				)
-				(justify left top)
-			)
-		)
-		(instances
-			(project "Logger"
-				(path "/2dac91f6-5de1-492e-9a04-36ab71ef854f"
-					(page "7")
-				)
-			)
-		)
-	)
-	(sheet
-		(at 175.26 97.79)
+		(at 68.58 85.09)
 		(size 12.7 3.81)
 		(fields_autoplaced yes)
@@
 		)
 		(property "Sheetname" "PowerSupply"
-			(at 175.26 97.1545 0)
+			(at 68.58 84.4545 0)
 			(effects
 				(font
@@
 		)
 		(property "Sheetfile" "PowerSupply.kicad_sch"
-			(at 175.26 102.1085 0)
+			(at 68.58 89.4085 0)
 			(effects
 				(font
@@
 		)
 		(instances
-			(project "Logger"
+			(project "MainBoard"
 				(path "/2dac91f6-5de1-492e-9a04-36ab71ef854f"
 					(page "5")
 				)
 			)
+		)
+	)
+	(sheet
+		(at 119.38 101.6)
+		(size 12.7 3.81)
+		(fields_autoplaced yes)
+		(stroke
+			(width 0.1524)
+			(type solid)
+		)
+		(fill
+			(color 0 0 0 0.0000)
+		)
+		(property "Sheetname" "ModuleConnector2"
+			(at 119.38 100.8884 0)
+			(effects
+				(font
+					(size 1.27 1.27)
+				)
+				(justify left bottom)
+			)
+		)
+		(property "Sheetfile" "ModuleConnector2.kicad_sch"
+			(at 119.38 105.9946 0)
+			(effects
+				(font
+					(size 1.27 1.27)
+				)
+				(justify left top)
+			)
+		)
+		(instances
+			(project "MainBoard"
+				(path "/2dac91f6-5de1-492e-9a04-36ab71ef854f"
+					(page "5")
+				)
+			)
+		)
+	)
+	(sheet
+		(at 114.3 85.09)
+		(size 12.7 3.81)
+		(fields_autoplaced yes)
+		(stroke
+			(width 0.1524)
+			(type solid)
+		)
+		(fill
+			(color 0 0 0 0.0000)
+		)
+		(property "Sheetname" "ModuleConnector1"
+			(at 114.3 84.3784 0)
+			(effects
+				(font
+					(size 1.27 1.27)
+				)
+				(justify left bottom)
+			)
+		)
+		(property "Sheetfile" "ModuleConnector1.kicad_sch"
+			(at 114.3 89.4846 0)
+			(effects
+				(font
+					(size 1.27 1.27)
+				)
+				(justify left top)
+			)
+		)
+		(instances
+			(project "MainBoard"
+				(path "/2dac91f6-5de1-492e-9a04-36ab71ef854f"
+					(page "3")
+				)
+			)
+		)
+	)
+	(sheet
+		(at 63.5 125.73)
+		(size 12.7 3.81)
+		(fields_autoplaced yes)
+		(stroke
+			(width 0.1524)
+			(type solid)
+		)
+		(fill
+			(color 0 0 0 0.0000)
+		)
+		(property "Sheetname" "Breadboard"
+			(at 63.5 125.0184 0)
+			(effects
+				(font
+					(size 1.27 1.27)
+				)
+				(justify left bottom)
+			)
+		)
+		(property "Sheetfile" "Breadboard.kicad_sch"
+			(at 63.5 130.1246 0)
+			(effects
+				(font
+					(size 1.27 1.27)
+				)
+				(justify left top)
+			)
+		)
+		(property "Field2" ""
+			(at 63.5 125.73 0)
+			(effects
+				(font
+					(size 1.27 1.27)
+				)
+				(hide yes)
+			)
+		)
+		(instances
+			(project "MainBoard"
+				(path "/2dac91f6-5de1-492e-9a04-36ab71ef854f"
+					(page "6")
+				)
+			)
+		)
+	)
+	(sheet
+		(at 80.01 104.14)
+		(size 12.7 3.81)
+		(fields_autoplaced yes)
+		(stroke
+			(width 0.1524)
+			(type solid)
+		)
+		(fill
+			(color 0 0 0 0.0000)
+		)
+		(property "Sheetname" "Mechanic"
+			(at 80.01 103.4284 0)
+			(effects
+				(font
+					(size 1.27 1.27)
+				)
+				(justify left bottom)
+			)
+		)
+		(property "Sheetfile" "Mechanic.kicad_sch"
+			(at 80.01 108.5346 0)
+			(effects
+				(font
+					(size 1.27 1.27)
+				)
+				(justify left top)
+			)
+		)
+		(instances
+			(project "MainBoard"
+				(path "/2dac91f6-5de1-492e-9a04-36ab71ef854f"
+					(page "4")
+				)
+			)
