File: Hardware/MainBoard/ModuleConnector.kicad_sch (KiCad schematic)
At the start: 2 parts, among them J1 Conn_02x20_Odd_Even

Commit message: draft of mainboard
Parts:
- added J10, J2, J3, J4, J6, J7, J8, J9: Conn_02x20_Odd_Even, Connector_PinSocket_2.54mm:PinSocket_2x20_P2.54mm_Vertical, symbol Connector_Generic:Conn_02x20_Odd_Even
- added TP10, TP11, TP12, TP13, TP14, TP15, TP16, TP17, TP18, TP19, TP2, TP20, TP21, TP22, TP23, TP24, TP25, TP26, TP27, TP28, TP29, TP3, TP30, TP31, TP32, TP33, TP34, TP35, TP36, TP37, TP38, TP39, TP4, TP40, TP5, TP6, TP7, TP8, TP9: TestPoint, TestPoint:TestPoint_Pad_D1.5mm, symbol Connector:TestPoint
Connections:
- net -12V: now also J10.5 (Pin_5), J2.5 (Pin_5), J3.5 (Pin_5), J4.5 (Pin_5), J6.5 (Pin_5), J7.5 (Pin_5), J8.5 (Pin_5), J9.5 (Pin_5)
- net -3V3: now also J10.3 (Pin_3), J2.3 (Pin_3), J3.3 (Pin_3), J4.3 (Pin_3), J6.3 (Pin_3), J7.3 (Pin_3), J8.3 (Pin_3), J9.3 (Pin_3)
- net -5V: now also J10.1 (Pin_1), J2.1 (Pin_1), J3.1 (Pin_1), J4.1 (Pin_1), J6.1 (Pin_1), J7.1 (Pin_1), J8.1 (Pin_1), J9.1 (Pin_1)
- net 12V: now also J10.6 (Pin_6), J2.6 (Pin_6), J3.6 (Pin_6), J4.6 (Pin_6), J6.6 (Pin_6), J7.6 (Pin_6), J8.6 (Pin_6), J9.6 (Pin_6)
- net 3V3: now also J10.4 (Pin_4), J2.4 (Pin_4), J3.4 (Pin_4), J4.4 (Pin_4), J6.4 (Pin_4), J7.4 (Pin_4), J8.4 (Pin_4), J9.4 (Pin_4)
- net 5V: now also J10.2 (Pin_2), J2.2 (Pin_2), J3.2 (Pin_2), J4.2 (Pin_2), J6.2 (Pin_2), J7.2 (Pin_2), J8.2 (Pin_2), J9.2 (Pin_2)
- net ANALOG1: now also J10.33 (Pin_33), J2.33 (Pin_33), J3.33 (Pin_33), J4.33 (Pin_33), J6.33 (Pin_33), J7.33 (Pin_33), J8.33 (Pin_33), J9.33 (Pin_33)
- net ANALOG2: now also J10.34 (Pin_34), J2.34 (Pin_34), J3.34 (Pin_34), J4.34 (Pin_34), J6.34 (Pin_34), J7.34 (Pin_34), J8.34 (Pin_34), J9.34 (Pin_34)
- net ANALOG3: now also J10.35 (Pin_35), J2.35 (Pin_35), J3.35 (Pin_35), J4.35 (Pin_35), J6.35 (Pin_35), J7.35 (Pin_35), J8.35 (Pin_35), J9.35 (Pin_35)
- net GND: now also J10.23 (Pin_23), J10.24 (Pin_24), J10.31 (Pin_31), J10.32 (Pin_32), J10.36 (Pin_36), J10.7 (Pin_7), J10.8 (Pin_8), J2.23 (Pin_23), J2.24 (Pin_24), J2.31 (Pin_31), J2.32 (Pin_32), J2.36 (Pin_36), J2.7 (Pin_7), J2.8 (Pin_8), J3.23 (Pin_23), J3.24 (Pin_24), J3.31 (Pin_31), J3.32 (Pin_32), J3.36 (Pin_36), J3.7 (Pin_7), J3.8 (Pin_8), J4.23 (Pin_23), J4.24 (Pin_24), J4.31 (Pin_31), J4.32 (Pin_32), J4.36 (Pin_36), J4.7 (Pin_7), J4.8 (Pin_8), J6.23 (Pin_23), J6.24 (Pin_24), J6.31 (Pin_31), J6.32 (Pin_32), J6.36 (Pin_36), J6.7 (Pin_7), J6.8 (Pin_8), J7.23 (Pin_23), J7.24 (Pin_24), J7.31 (Pin_31), J7.32 (Pin_32), J7.36 (Pin_36), J7.7 (Pin_7), J7.8 (Pin_8), J8.23 (Pin_23), J8.24 (Pin_24), J8.31 (Pin_31), J8.32 (Pin_32), J8.36 (Pin_36), J8.7 (Pin_7), J8.8 (Pin_8), J9.23 (Pin_23), J9.24 (Pin_24), J9.31 (Pin_31), J9.32 (Pin_32), J9.36 (Pin_36), J9.7 (Pin_7), J9.8 (Pin_8)
- net GPIO1: now also J10.9 (Pin_9), J2.9 (Pin_9), J3.9 (Pin_9), J4.9 (Pin_9), J6.9 (Pin_9), J7.9 (Pin_9), J8.9 (Pin_9), J9.9 (Pin_9)
- net GPIO10: now also J10.18 (Pin_18), J2.18 (Pin_18), J3.18 (Pin_18), J4.18 (Pin_18), J6.18 (Pin_18), J7.18 (Pin_18), J8.18 (Pin_18), J9.18 (Pin_18)
- net GPIO11: now also J10.19 (Pin_19), J2.19 (Pin_19), J3.19 (Pin_19), J4.19 (Pin_19), J6.19 (Pin_19), J7.19 (Pin_19), J8.19 (Pin_19), J9.19 (Pin_19)
- net GPIO12: now also J10.20 (Pin_20), J2.20 (Pin_20), J3.20 (Pin_20), J4.20 (Pin_20), J6.20 (Pin_20), J7.20 (Pin_20), J8.20 (Pin_20), J9.20 (Pin_20)
- net GPIO2: now also J10.10 (Pin_10), J2.10 (Pin_10), J3.10 (Pin_10), J4.10 (Pin_10), J6.10 (Pin_10), J7.10 (Pin_10), J8.10 (Pin_10), J9.10 (Pin_10)
- net GPIO3: now also J10.11 (Pin_11), J2.11 (Pin_11), J3.11 (Pin_11), J4.11 (Pin_11), J6.11 (Pin_11), J7.11 (Pin_11), J8.11 (Pin_11), J9.11 (Pin_11)
- net GPIO4: now also J10.12 (Pin_12), J2.12 (Pin_12), J3.12 (Pin_12), J4.12 (Pin_12), J6.12 (Pin_12), J7.12 (Pin_12), J8.12 (Pin_12), J9.12 (Pin_12)
- net GPIO5: now also J10.13 (Pin_13), J2.13 (Pin_13), J3.13 (Pin_13), J4.13 (Pin_13), J6.13 (Pin_13), J7.13 (Pin_13), J8.13 (Pin_13), J9.13 (Pin_13)
- net GPIO6: now also J10.14 (Pin_14), J2.14 (Pin_14), J3.14 (Pin_14), J4.14 (Pin_14), J6.14 (Pin_14), J7.14 (Pin_14), J8.14 (Pin_14), J9.14 (Pin_14)
- net GPIO7: now also J10.15 (Pin_15), J2.15 (Pin_15), J3.15 (Pin_15), J4.15 (Pin_15), J6.15 (Pin_15), J7.15 (Pin_15), J8.15 (Pin_15), J9.15 (Pin_15)
- net GPIO8: now also J10.16 (Pin_16), J2.16 (Pin_16), J3.16 (Pin_16), J4.16 (Pin_16), J6.16 (Pin_16), J7.16 (Pin_16), J8.16 (Pin_16), J9.16 (Pin_16)
- net GPIO9: now also J10.17 (Pin_17), J2.17 (Pin_17), J3.17 (Pin_17), J4.17 (Pin_17), J6.17 (Pin_17), J7.17 (Pin_17), J8.17 (Pin_17), J9.17 (Pin_17)
- net I2C_SCL: now also J10.21 (Pin_21), J2.21 (Pin_21), J3.21 (Pin_21), J4.21 (Pin_21), J6.21 (Pin_21), J7.21 (Pin_21), J8.21 (Pin_21), J9.21 (Pin_21)
- net I2C_SDA: now also J10.22 (Pin_22), J2.22 (Pin_22), J3.22 (Pin_22), J4.22 (Pin_22), J6.22 (Pin_22), J7.22 (Pin_22), J8.22 (Pin_22), J9.22 (Pin_22)
- net SPI_CS1: now also J10.28 (Pin_28), J2.28 (Pin_28), J3.28 (Pin_28), J4.28 (Pin_28), J6.28 (Pin_28), J7.28 (Pin_28), J8.28 (Pin_28), J9.28 (Pin_28)
- net SPI_CS2: now also J10.29 (Pin_29), J2.29 (Pin_29), J3.29 (Pin_29), J4.29 (Pin_29), J6.29 (Pin_29), J7.29 (Pin_29), J8.29 (Pin_29), J9.29 (Pin_29)
- net SPI_CS3: now also J10.30 (Pin_30), J2.30 (Pin_30), J3.30 (Pin_30), J4.30 (Pin_30), J6.30 (Pin_30), J7.30 (Pin_30), J8.30 (Pin_30), J9.30 (Pin_30)
- net SPI_MISO: now also J10.27 (Pin_27), J2.27 (Pin_27), J3.27 (Pin_27), J4.27 (Pin_27), J6.27 (Pin_27), J7.27 (Pin_27), J8.27 (Pin_27), J9.27 (Pin_27)
- net SPI_MOSI: now also J10.26 (Pin_26), J2.26 (Pin_26), J3.26 (Pin_26), J4.26 (Pin_26), J6.26 (Pin_26), J7.26 (Pin_26), J8.26 (Pin_26), J9.26 (Pin_26)
- net SPI_SCLK: now also J10.25 (Pin_25), J2.25 (Pin_25), J3.25 (Pin_25), J4.25 (Pin_25), J6.25 (Pin_25), J7.25 (Pin_25), J8.25 (Pin_25), J9.25 (Pin_25)
- net UART1_RX: now also J10.38 (Pin_38), J2.38 (Pin_38), J3.38 (Pin_38), J4.38 (Pin_38), J6.38 (Pin_38), J7.38 (Pin_38), J8.38 (Pin_38), J9.38 (Pin_38)
- net UART1_TX: now also J10.37 (Pin_37), J2.37 (Pin_37), J3.37 (Pin_37), J4.37 (Pin_37), J6.37 (Pin_37), J7.37 (Pin_37), J8.37 (Pin_37), J9.37 (Pin_37)
- net UART2_RX: now also J10.40 (Pin_40), J2.40 (Pin_40), J3.40 (Pin_40), J4.40 (Pin_40), J6.40 (Pin_40), J7.40 (Pin_40), J8.40 (Pin_40), J9.40 (Pin_40)
- net UART2_TX: now also J10.39 (Pin_39), J2.39 (Pin_39), J3.39 (Pin_39), J4.39 (Pin_39), J6.39 (Pin_39), J7.39 (Pin_39), J8.39 (Pin_39), J9.39 (Pin_39)
Other:
- moved on the sheet: J1, TP1
