File: Hardware/DataAcquisitionUnit/PowerSupply.kicad_sch (KiCad schematic)
At the start: 10 parts, among them U1 LM2901, U2 LD1117S50TR_SOT223

Commit message: hw 4.1 pcb, ci rework
Parts:
- C11, C13: value 100n -> 330n
- C12: value 1u -> 330n
- U2: footprint Package_TO_SOT_SMD:SOT-223 -> Package_TO_SOT_SMD:SOT-223-3_TabPin2
Changed lines of the file:
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@@
 			)
 		)
-		(property "Value" "1u"
+		(property "Value" "330n"
 			(at 156.591 105.283 0)
 			(effects
@@
 			)
 		)
-		(property "Footprint" "Package_TO_SOT_SMD:SOT-223"
+		(property "Footprint" "Package_TO_SOT_SMD:SOT-223-3_TabPin2"
 			(at 121.92 90.17 0)
 			(effects
@@
 			)
 		)
-		(property "Value" "100n"
+		(property "Value" "330n"
 			(at 168.021 105.283 0)
 			(effects
@@
 			)
 		)
-		(property "Value" "100n"
+		(property "Value" "330n"
 			(at 109.601 105.283 0)
 			(effects
