File: Hardware/DataAcquisitionUnit/PulseCounter.kicad_sch (KiCad schematic)
At the start: 45 parts, among them J1 Conn_Coaxial, J2 Conn_Coaxial, J3 Conn_Coaxial, J4 Conn_Coaxial, U1 LM2901

Commit message: hw 4.1 pcb, ci rework
Parts:
- removed C3, C4, C7, C8: 100n, Capacitor_SMD:C_0805_2012Metric, symbol Device:C
- added D10, D6, D7, D9: PJGBLC03C_R1_00001, Diode_SMD:D_SOD-323F, symbol Device:D_TVS
- R10, R19, R20, R9: value 1k -> 10k
- R13, R14, R3, R4: value 510k -> 8k2
- R15, R16, R17, R18, R5, R6, R7, R8: value 0R -> TBD
- RV1, RV2, RV3, RV4: footprint Potentiometer_THT:Potentiometer_Bourns_3296W_Vertical -> Potentiometer_THT:Potentiometer_Bourns_3296Y_Vertical
Connections:
- net GND: now also D10.1 (A1), D6.1 (A1), D7.1 (A1), D9.1 (A1)
- net at C2.1, R2.2, R4.2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: now also D6.2 (A2)
- net at C5.1, R11.2, R13.2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: now also D9.2 (A2)
- net at C1.1, R1.2, R3.2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: now also D7.2 (A2)
- net at C6.1, R12.2, R14.2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: now also D10.2 (A2)
Other:
- moved on the sheet: C1, C5, C6, J1, J2, J3, J4, R1, R11, R12, R13, R14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
