File: Hardware/DataAcquisitionUnit/UART.kicad_sch (KiCad schematic)
At the start: 9 parts, among them J10 DE9_Pins_MountingHoles, J11 DE9_Pins_MountingHoles, J9 DE9_Pins_MountingHoles

Commit message: hw 4.1 pcb, ci rework
Parts:
- added D1, D2, D3, D4, D5, D8: PJGBLC03C_R1_00001, Diode_SMD:D_SOD-323F, symbol Device:D_TVS
Connections:
- net GND: now also J10.5, J11.5, J9.5, D1.1 (A1), D2.1 (A1), D3.1 (A1), D4.1 (A1), D5.1 (A1), D8.1 (A1)
- net USART1_RX: now also D3.2 (A2)
- net USART1_TX: now also D2.2 (A2)
- net USART2_RX: now also D5.2 (A2)
- net USART2_TX: now also D4.2 (A2)
- net USART3_RX: now also D8.2 (A2)
- net USART3_TX: now also D1.2 (A2)
- no-connect marks 21 -> 18
Other:
- moved on the sheet: J10, R23, R24
