File: Hardware/DataProcessingUnit/ExtensionConnectors.kicad_sch (KiCad schematic)
At the start: 1 part

Commit message: hw 4.1 pcb, ci rework
Connections:
- net 5V: no longer J5.39 (Pin_39)
- net -12V: no longer names the net of J5.36 (Pin_36)
- net -12V: no longer J5.56 (Pin_56)
- net -3V3: no longer names the net of J5.38 (Pin_38)
- net -3V3: no longer J5.58 (Pin_58)
- net -5V: no longer names the net of J5.40 (Pin_40)
- net -5V: no longer J5.60 (Pin_60)
- net 12V: no longer names the net of J5.35 (Pin_35)
- net 12V: no longer J5.55 (Pin_55)
- net 3V3_FROM_MAINBOARD: no longer names the net of J5.37 (Pin_37)
- net 3V3_FROM_MAINBOARD: no longer J5.57 (Pin_57)
- net BOOT0 renamed GPIO_24
- net NRST: no longer names the net of J5.41 (Pin_41)
- no-connect marks 0 -> 12
