File: Hardware/DataProcessingUnit/DataProcessingUnit.kicad_pcb (KiCad board)
At the start: 2 copper layers, 85 x 50 mm, 50 parts, among them J2 USB_B_Micro, J3 Conn_02x05_Odd_Even, Q2 BC847, SW1 SW_Push, U2 LD1117S33TR, U3 STM32F103RBTx, Y1 32,768kHz, Y2 Crystal

Commit message: hw 4.1 integration
Parts:
- C11, C12: value 6p8 -> 18p
- C13, C14: value 6p8 -> 22p
- R13, R14: value TBD -> 0R
- Y2: value Crystal -> 8M
Changed lines of the file:
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@@
 			)
 		)
-		(property "Value" "6p8"
+		(property "Value" "18p"
 			(at 0 1.679999 135)
 			(layer "F.Fab")
@@
 			)
 		)
-		(property "Value" "TBD"
+		(property "Value" "0R"
 			(at 0 1.65 45)
 			(layer "F.Fab")
@@
 			)
 		)
-		(property "Value" "TBD"
+		(property "Value" "0R"
 			(at 0 1.65 45)
 			(layer "F.Fab")
@@
 			)
 		)
-		(property "Value" "Crystal"
+		(property "Value" "8M"
 			(at 0 3.55 135)
 			(layer "F.Fab")
@@
 			)
 		)
-		(property "Value" "6p8"
+		(property "Value" "18p"
 			(at 0 1.679999 135)
 			(layer "F.Fab")
@@
 			)
 		)
-		(property "Value" "6p8"
+		(property "Value" "22p"
 			(at 0 1.679999 45)
 			(layer "F.Fab")
@@
 			)
 		)
-		(property "Value" "6p8"
+		(property "Value" "22p"
 			(at 0 1.679999 45)
 			(layer "F.Fab")
