File: Hardware/HumanMachineInterface/HumanMachineInterface.kicad_pcb (KiCad board)
At the start: 2 copper layers, 85 x 60 mm, 22 parts, among them Q1 Q_Photo_NPN, SW1 SW_Push, SW2 SW_Push, SW3 SW_Push, SW4 SW_Push, U2 ST7735S

Commit message: hw 4.1 pcb, ci rework
Parts:
- removed JP1: Jumper_2_Small_Open, Jumper:SolderJumper-2_P1.3mm_Open_TrianglePad1.0x1.5mm
- added C4: 4u7, Capacitor_SMD:C_0805_2012Metric, B.Cu at (163.2, 79.0)
- added JP2: SolderJumper_2_Bridged, Jumper:SolderJumper-2_P1.3mm_Bridged_Pad1.0x1.5mm, B.Cu at (208.8, 108.0)
- added R5: 1M, Resistor_SMD:R_0805_2012Metric, B.Cu at (164.4, 107.4)
- added R6: 1M, Resistor_SMD:R_0805_2012Metric, B.Cu at (168.0, 107.4)
- added R7: 1M, Resistor_SMD:R_0805_2012Metric, B.Cu at (171.5, 107.4)
- added TP7: TestPoint, TestPoint:TestPoint_Pad_D1.5mm, B.Cu at (205.5, 108.0)
- added TP8: TestPoint, TestPoint:TestPoint_Pad_D1.5mm, B.Cu at (196.2, 109.8)
- C1: value 330n -> 4u7
- R1: value 2M -> 1M
- SW1, SW2, SW3, SW4: footprint Button_Switch_SMD:SW_SPST_PTS645 -> Button_Switch_SMD:SW_SPST_PTS645Sx43SMTR92
- moved C2 12.0 mm to (163.2, 83.5), turned to 0 degrees
- moved C1 8.99 mm to (163.2, 81.2), turned to 0 degrees
- moved U2 8.78 mm to (158.5, 70.2)
- moved SW1 8.58 mm to (140.0, 74.0)
- moved G*** 8.44 mm to (132.5, 74.0)
- moved TP1 7.18 mm to (155.0, 96.5)
- moved TP2 7.09 mm to (155.0, 93.8)
- moved TP3 6.96 mm to (155.0, 91.0)
- moved TP4 6.77 mm to (155.0, 88.2)
- moved SW2 6.71 mm to (140.0, 84.0)
- moved TP5 6.58 mm to (155.0, 85.4)
- moved G*** 6.52 mm to (132.5, 84.0)
- moved TP6 6.39 mm to (155.0, 82.6)
- moved SW3 4.94 mm to (140.0, 94.0)
- moved G*** 4.69 mm to (132.5, 94.0)
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Connections:
- J5 pad 13: GPIO_4 -> unconnected-(J5-Pin_13-Pad13)
- J5 pad 5: unconnected-(J5-Pin_5-Pad5) -> GPIO_12
- J5 pad 7: GPIO_10 -> unconnected-(J5-Pin_7-Pad7)
- J5 pad 9: unconnected-(J5-Pin_9-Pad9) -> GPIO_8
- R1 pad 1: 3V3_FROM_MAINBOARD -> Net-(R1-Pad1)
- TP2 pad 1: GPIO_10 -> GPIO_12
- TP4 pad 1: GPIO_4 -> GPIO_8
- U2 pad 5: GPIO_4 -> GPIO_8
- U2 pad 7: GPIO_10 -> GPIO_12
Routing:
- net 3V3_FROM_MAINBOARD: track 108.3 -> 59.7 mm
- net GPIO_8: track 0.00 -> 45.8 mm
- net GPIO_4: track 42.1 -> 0.00 mm
- net GPIO_12: track 0.00 -> 37.3 mm
- net Net-(JP2-B): track 26.5 -> 63.0 mm
- net GPIO_10: track 36.3 -> 0.00 mm
- net GND: track 16.7 -> 2.54 mm, vias 16 -> 18
- net SPI1_SCK: track 43.5 -> 52.5 mm
- net GPIO_15: track 54.8 -> 46.6 mm
- net SPI1_MOSI: track 47.9 -> 41.2 mm
- net GPIO_16: track 45.8 -> 39.7 mm
- net GPIO_5: track 35.6 -> 30.5 mm
- net GPIO_6: track 32.9 -> 30.2 mm
- net GPIO_13: track 29.9 -> 27.4 mm
- net GPIO_18: track 54.3 -> 56.6 mm
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Other:
- board size 85 x 60 mm -> 85 x 50 mm
- board text added: "HumanMachineInterface rev 1.1"
- board text removed: "HumanMachineInterface rev 1.0"
