File: Hardware/HumanMachineInterface/HumanMachineInterface.kicad_sch (KiCad schematic)
At the start: 18 parts, among them Q1 Q_Photo_NPN, SW1 SW_Push, SW2 SW_Push, SW3 SW_Push, SW4 SW_Push, U2 ST7735S

Commit message: hw 4.1 pcb, ci rework
Parts:
- removed JP1: Jumper_2_Small_Open, Jumper:SolderJumper-2_P1.3mm_Open_TrianglePad1.0x1.5mm, symbol Jumper:Jumper_2_Small_Open
- added C4: 4u7, Capacitor_SMD:C_0805_2012Metric, symbol Device:C
- added JP2: SolderJumper_2_Bridged, Jumper:SolderJumper-2_P1.3mm_Bridged_Pad1.0x1.5mm, symbol Jumper:SolderJumper_2_Bridged
- added R5, R6, R7: 1M, Resistor_SMD:R_0805_2012Metric, symbol Device:R
- added TP7, TP8: TestPoint, TestPoint:TestPoint_Pad_D1.5mm, symbol Connector:TestPoint
- C1: value 330n -> 4u7
- R1: value 2M -> 1M
- SW1, SW2, SW3, SW4: footprint Button_Switch_SMD:SW_SPST_PTS645 -> Button_Switch_SMD:SW_SPST_PTS645Sx43SMTR92
Connections:
- net 3V3_FROM_MAINBOARD: now also JP2.1 (A), R7.1; no longer R1.1
- net GND: now also C4.2
- net GPIO_18: now also TP8.1
- net at C1.1, C2.1, U2.2 (VCC): now also C4.1, JP2.2 (B), TP7.1
- net GPIO_12: now reaches J5.5 (Pin_5)
- net GPIO_12: now also TP2.1, U2.7 (CS)
- net GPIO_8: now reaches J5.9 (Pin_9)
- net GPIO_8: now also TP4.1, U2.5 (RES)
- removed net GPIO_10: J5.7 (Pin_7), TP2.1, U2.7 (CS)
- removed net GPIO_4: J5.13 (Pin_13), TP4.1, U2.5 (RES)
- new net: R6.1, R7.2
- new net: R1.1, R5.2
- new net: R5.1, R6.2
Other:
- moved on the sheet: C1, C2, TP1, TP2, TP3, TP4, TP5, TP6, U2

Commit message: hw 4.1 integration
Parts:
- C3: value 330n -> 100n
- R1, R5, R6, R7: value 1M -> 510k
Changed lines of the file:
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@@
 			)
 		)
-		(property "Value" "1M"
+		(property "Value" "510k"
 			(at 171.958 96.393 0)
 			(effects
@@
 			)
 		)
-		(property "Value" "1M"
+		(property "Value" "510k"
 			(at 171.958 123.063 0)
 			(effects
@@
 			)
 		)
-		(property "Value" "1M"
+		(property "Value" "510k"
 			(at 171.958 105.283 0)
 			(effects
@@
 			)
 		)
-		(property "Value" "1M"
+		(property "Value" "510k"
 			(at 171.958 114.173 0)
 			(effects
@@
 		(fields_autoplaced yes)
 		(property "Reference" "C3"
-			(at 193.4211 132.4415 0)
-			(effects
-				(font
-					(size 1.27 1.27)
-				)
-				(justify left)
-			)
-		)
-		(property "Value" "330n"
-			(at 193.4211 135.2166 0)
-			(effects
-				(font
+			(at 194.31 132.0799 0)
+			(effects
+				(font
+					(size 1.27 1.27)
+				)
+				(justify left)
+			)
+		)
+		(property "Value" "100n"
+			(at 194.31 134.6199 0)
+			(effects
+				(font
